File: Kicad/Bat_IMU_nRF5340/Bat_IMU_nRF5340.kicad_pcb (KiCad board)
At the start: 2 copper layers, 9 parts, among them J1 FTSH-105-01-F-DV-P-TR, J2 MEM2075-00-140-01-A, U1 BT40F, U2 LP2985-3.3, U3 ICM-42688-P

Commit message: Kicad first version layout update
Parts:
- removed U2: LP2985-3.3, Package_TO_SOT_SMD:SOT-23-5
- added C4: C, Capacitor_SMD:C_0603_1608Metric, F.Cu at (124.8, 74.4)
- added C5: C, Capacitor_SMD:C_0603_1608Metric, F.Cu at (129.5, 85.1)
- added C6: C, Capacitor_SMD:C_0603_1608Metric, F.Cu at (143.2, 80.0)
- added Q1: PMOS, Package_TO_SOT_SMD:SOT-89-3_Handsoldering, F.Cu at (105.7, 69.4)
- added Q2: NMOS, Package_TO_SOT_SMD:SOT-89-3_Handsoldering, F.Cu at (110.8, 69.4)
- added R1: 100k, Resistor_SMD:R_0603_1608Metric_Pad0.98x0.95mm_HandSolder, F.Cu at (105.7, 63.8)
- added R2: R, Resistor_SMD:R_0603_1608Metric_Pad0.98x0.95mm_HandSolder, F.Cu at (110.5, 64.0)
- added R3: R, Resistor_SMD:R_0603_1608Metric_Pad0.98x0.95mm_HandSolder, F.Cu at (110.5, 62.5)
- moved MK1 25.7 mm to (127.2, 73.9)
- moved C1 19.7 mm to (143.0, 85.0)
- moved C2 19.7 mm to (140.0, 86.0)
- moved C3 19.7 mm to (140.0, 84.0)
- moved J1 14.0 mm to (135.0, 64.5)
- moved U3 7.63 mm to (121.5, 73.0), turned to 90 degrees
- moved U1 4.27 mm to (114.1, 71.0)
- moved J2 3.48 mm to (116.3, 84.3)
Connections:
- net /CS renamed /SPI3_CS
- net /DI renamed /SPI3_MOSI
- net /DO renamed /SPI3_MISO
- net /SCK renamed /SPI3_SCK
- C1 pad 1: VIN -> GND
- C1 pad 2: GND -> VBAT
- C2 pad 1: Net-(U2-BP) -> GND
- C2 pad 2: GND -> VCC
- C3 pad 1: VCC -> GND
- C3 pad 2: GND -> VCC
- J1 pad 08: unconnected-(J1-Pad08) -> /SWD_NC
- U1 pad P$C6: unconnected-(U1-C6/P025-PadP$C6) -> /SPI2_INT
- U1 pad P$D1: unconnected-(U1-D1/P026-PadP$D1) -> /ICM_CLKIN
- U1 pad P$D2: unconnected-(U1-D2/P027-PadP$D2) -> /SWD_NC
- U1 pad P$D3: unconnected-(U1-D3/P028-PadP$D3) -> VBAT_div
- U1 pad P$D4: unconnected-(U1-D4/P029-PadP$D4) -> Net-(Q2-G)
- U1 pad P$F4: VCC -> VBAT
- U1 pad P$Z2: unconnected-(U1-Z2/P111-PadP$Z2) -> /I2S_SDIN
- U1 pad P$Z4: /I2S_SDIN -> unconnected-(U1-Z4/P113-PadP$Z4)
- U3 pad 4: unconnected-(U3-INT1/INT-Pad4) -> /SPI2_INT
- U3 pad 9: GND -> /ICM_CLKIN
Routing:
- net GND: track 0.00 -> 138.5 mm, vias 0 -> 5
- net VCC: track 0.00 -> 37.2 mm
- net VBAT: track 0.00 -> 30.0 mm, vias 0 -> 2
- net /SPI3_MOSI: track 0.00 -> 29.8 mm, vias 0 -> 2
- net /SPI3_SCK: track 0.00 -> 28.0 mm, vias 0 -> 2
- net /I2S_SCK_M: track 0.00 -> 23.9 mm, vias 0 -> 2
- net /SPI3_MISO: track 0.00 -> 22.8 mm, vias 0 -> 2
- net /SPI2_MOSI: track 0.00 -> 22.2 mm
- net /SPI3_CS: track 0.00 -> 22.0 mm, vias 0 -> 2
- net Net-(Q2-G): track 0.00 -> 20.6 mm, vias 0 -> 2
- net VBAT_div: track 0.00 -> 20.5 mm, vias 0 -> 2
- net /I2S_SDIN: track 0.00 -> 17.8 mm, vias 0 -> 2
- net Net-(Q1-G): track 0.00 -> 17.7 mm
- net /SWD_NC: track 0.00 -> 17.6 mm
- net /SPI2_SCK: track 0.00 -> 13.5 mm
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
Commit message: Kicad PCB update
Parts:
- removed C4, C5, C6: C, Capacitor_SMD:C_0603_1608Metric
- added Battery: ~, Bat_tag_Library:Battery_entry, F.Cu at (128.3, 81.9)
- added C7: C, Capacitor_SMD:C_0603_1608Metric, F.Cu at (133.5, 79.2)
- added I2S_debug1: ~, Bat_tag_Library:I2S_debug, F.Cu at (112.6, 84.8)
- added REF**: Mecha_Pad, Bat_tag_Library:Mecha_Pad, F.Cu at (107.2, 68.6)
- added REF**: Mecha_Pad, Bat_tag_Library:Mecha_Pad, F.Cu at (132.3, 68.6)
- added REF**: Mecha_Pad, Bat_tag_Library:Mecha_Pad, F.Cu at (132.3, 82.8)
- added REF**: Mecha_Pad, Bat_tag_Library:Mecha_Pad, F.Cu at (107.2, 82.8)
- added SPI_debug1: ~, Bat_tag_Library:SPI_debug, F.Cu at (121.0, 84.8)
- J2: moved to B.Cu
- Q1, Q2: footprint Package_TO_SOT_SMD:SOT-89-3_Handsoldering -> Package_TO_SOT_SMD:SOT-89-3
- moved R1 22.6 mm to (127.8, 68.5)
- moved C2 21.8 mm to (118.7, 81.2), turned to 90 degrees
- moved C1 21.5 mm to (129.3, 68.5), turned to 90 degrees
- moved R3 18.9 mm to (112.8, 81.3), turned to -90 degrees
- moved R2 17.3 mm to (111.3, 81.3), turned to 90 degrees
- moved J2 16.8 mm to (117.8, 67.7), turned to 0 degrees
- moved MK1 13.4 mm to (116.3, 81.6)
- moved C3 12.5 mm to (128.8, 78.5)
- moved J1 10.6 mm to (130.6, 74.2)
- moved Q2 9.21 mm to (108.2, 78.2), turned to 0 degrees
- moved U3 8.74 mm to (122.7, 81.7), turned to 180 degrees
- moved U1 8.72 mm to (111.7, 79.4)
- moved Q1 4.51 mm to (108.2, 73.2), turned to 0 degrees
Connections:
- J2 pad SH1: unconnected-(J2-SHIELD-PadSH1) -> GND
- J2 pad SH2: unconnected-(J2-SHIELD-PadSH1) -> GND
- J2 pad SH3: unconnected-(J2-SHIELD-PadSH1) -> GND
- J2 pad SH4: unconnected-(J2-SHIELD-PadSH1) -> GND
Routing:
- net GND: track 138.5 -> 176.2 mm, vias 5 -> 15
- net VBAT: track 30.0 -> 63.5 mm, vias 2 -> 3
- net /SPI2_SCK: track 13.5 -> 33.4 mm, vias 0 -> 2
- net /SPI3_CS: track 22.0 -> 5.60 mm, vias 2 -> 1
- net /SPI2_MISO: track 12.5 -> 24.9 mm, vias 0 -> 4
- net VCC: track 37.2 -> 25.9 mm, vias 0 -> 1
- net Net-(Q1-G): track 17.7 -> 27.6 mm
- net /SPI2_CS: track 12.1 -> 19.9 mm, vias 2 -> 4
- net /SPI3_MOSI: track 29.8 -> 36.7 mm, vias 2 -> 1
- net /SPI3_MISO: track 22.8 -> 28.6 mm, vias 2 -> 1
- net VBAT_div: track 20.5 -> 15.4 mm
- net Net-(Q2-G): track 20.6 -> 25.2 mm
- net /I2S_SDIN: track 17.8 -> 13.3 mm, vias 2 -> 0
- net /ICM_CLKIN: track 8.31 -> 12.4 mm, vias 0 -> 2
- net /SPI2_INT: track 9.26 -> 13.3 mm
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- added copper zone on B.Cu, net GND
- added copper zone on F.Cu, net GND
Other:
- board outline added: 29.2 x 18.3 mm
