File: Kicad/Bat_IMU_nRF5340/Bat_IMU_nRF5340.kicad_sch (KiCad schematic)
At the start: 9 parts, among them J1 FTSH-105-01-F-DV-P-TR, J2 MEM2075-00-140-01-A, U1 BT40F, U2 LP2985-3.3, U3 ICM-42688-P

Commit message: Kicad first version layout update
Parts:
- removed U2: LP2985-3.3, Package_TO_SOT_SMD:SOT-23-5, symbol Regulator_Linear:LP2985-3.3
- added C4, C5, C6: C, Capacitor_SMD:C_0603_1608Metric, symbol Device:C
- added Q1: PMOS, Package_TO_SOT_SMD:SOT-89-3_Handsoldering, symbol Simulation_SPICE:PMOS
- added Q2: NMOS, Package_TO_SOT_SMD:SOT-89-3_Handsoldering, symbol Simulation_SPICE:NMOS
- added R1: 100k, Resistor_SMD:R_0603_1608Metric_Pad0.98x0.95mm_HandSolder, symbol Device:R
- added R2, R3: R, Resistor_SMD:R_0603_1608Metric_Pad0.98x0.95mm_HandSolder, symbol Device:R
Connections:
- net VIN is gone; now on net GND: C1.1
- net GND: now also C2.1, C3.1, C4.1, C5.1, C6.1, Q2.3 (S), R3.2; no longer C1.2, C2.2, C3.2, U3.9 (INT2/FSYNC/CLKIN)
- net VCC: now also C2.2, C3.2, C4.2, C5.2, C6.2; no longer C3.1, U1.P$F4 (F4/VDDH)
- net ICM_CLKIN: now reaches U1.P$D1 (D1/P026)
- net ICM_CLKIN: now also U3.9 (INT2/FSYNC/CLKIN)
- net SWD_NC: now reaches U1.P$D2 (D2/P027)
- net SWD_NC: now also J1.08
- net VBAT_div: now reaches U1.P$D3 (D3/P028)
- net VBAT_div: now also R2.2, R3.1
- net at U1.P$D4 (D4/P029): now also Q2.2 (G)
- net CS renamed SPI3_CS
- net DI renamed SPI3_MOSI
- net DO renamed SPI3_MISO
- net SCK renamed SPI3_SCK
- new net: Q1.2 (G), Q2.1 (D), R1.1
- new net: Q1.3 (S), R2.1
- new net VBAT: C1.2, Q1.1 (D), R1.2, U1.P$F4 (F4/VDDH)
- no-connect marks 47 -> 42

Commit message: Kicad PCB update
Parts:
- added Battery_entry1: ~, Bat_tag_Library:Battery_entry, symbol Bat_tag_Library:Battery_entry
- added C7: C, Capacitor_SMD:C_0603_1608Metric, symbol Device:C
- added I2S_debug1: ~, Bat_tag_Library:I2S_debug, symbol Bat_tag_Library:I2S_debug
- added SPI_debug1: ~, Bat_tag_Library:SPI_debug, symbol Bat_tag_Library:SPI_debug
- Q1, Q2: footprint Package_TO_SOT_SMD:SOT-89-3_Handsoldering -> Package_TO_SOT_SMD:SOT-89-3
Connections:
- net GND: now also J2.SH1 (SHIELD), J2.SH2 (SHIELD), J2.SH3 (SHIELD), J2.SH4 (SHIELD), Battery_entry1.2, C7.1, SPI_debug1.1
- net I2S_SCK_M: now also I2S_debug1.1
- net I2S_SDIN: now also I2S_debug1.2
- net SPI2_CS: now also SPI_debug1.3
- net SPI2_INT: now also SPI_debug1.6
- net SPI2_MISO: now also SPI_debug1.5
- net SPI2_MOSI: now also SPI_debug1.4
- net SPI2_SCK: now also SPI_debug1.2
- net VBAT: now also Battery_entry1.1, C7.2
